File: Hardware/PCB/ringmod_2/ringmod_2.kicad_sch (KiCad schematic)
At the start: 15 parts, among them J10 2_pin_Molex_header, J11 2_pin_Molex_header, J12 3_pin_Molex_connector, J13 2_pin_Molex_connector, J14 2_pin_Molex_connector, J15 2_pin_Molex_connector, J6 AudioJack2, J7 3_pin_Molex_header, J8 2_pin_Molex_header

Commit message: Update pot symbols
Changed lines of the file:
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@@
   )
   (junction (at 115.57 91.44) (diameter 0) (color 0 0 0 0))
+  (junction (at 177.8 93.98) (diameter 0) (color 0 0 0 0))
+  (junction (at 166.37 85.09) (diameter 0) (color 0 0 0 0))
+  (junction (at 166.37 102.87) (diameter 0) (color 0 0 0 0))
   (junction (at 162.56 97.79) (diameter 0) (color 0 0 0 0))
-  (junction (at 177.8 93.98) (diameter 0) (color 0 0 0 0))
+  (junction (at 162.56 106.68) (diameter 0) (color 0 0 0 0))
+  (junction (at 161.29 88.9) (diameter 0) (color 0 0 0 0))
+  (junction (at 166.37 93.98) (diameter 0) (color 0 0 0 0))
+  (junction (at 166.37 110.49) (diameter 0) (color 0 0 0 0))
+  (junction (at 166.37 92.71) (diameter 0) (color 0 0 0 0))
   (junction (at 177.8 102.87) (diameter 0) (color 0 0 0 0))
-  (junction (at 161.29 88.9) (diameter 0) (color 0 0 0 0))
   (junction (at 166.37 101.6) (diameter 0) (color 0 0 0 0))
-  (junction (at 166.37 92.71) (diameter 0) (color 0 0 0 0))
-  (junction (at 166.37 102.87) (diameter 0) (color 0 0 0 0))
-  (junction (at 162.56 106.68) (diameter 0) (color 0 0 0 0))
-  (junction (at 166.37 93.98) (diameter 0) (color 0 0 0 0))
-  (junction (at 166.37 85.09) (diameter 0) (color 0 0 0 0))
-  (junction (at 166.37 110.49) (diameter 0) (color 0 0 0 0))
   (wire (pts (xy 166.37 85.09) (xy 181.61 85.09))
     (stroke (width 0) (type default) (color 0 0 0 0))
@@
     (stroke (width 0) (type default) (color 0 0 0 0))
   )
+  (polyline (pts (xy 137.16 67.31) (xy 137.16 123.19))
+    (stroke (width 0) (type default) (color 0 0 0 0))
+  )
+  (polyline (pts (xy 137.16 67.31) (xy 212.09 67.31))
+    (stroke (width 0) (type default) (color 0 0 0 0))
+  )
   (polyline (pts (xy 137.16 123.19) (xy 212.09 123.19))
     (stroke (width 0) (type default) (color 0 0 0 0))
   )
-  (polyline (pts (xy 137.16 67.31) (xy 212.09 67.31))
-    (stroke (width 0) (type default) (color 0 0 0 0))
-  )
-  (polyline (pts (xy 137.16 67.31) (xy 137.16 123.19))
-    (stroke (width 0) (type default) (color 0 0 0 0))
-  )
   (wire (pts (xy 113.03 86.36) (xy 118.11 86.36))
     (stroke (width 0) (type default) (color 0 0 0 0))
@@
     (stroke (width 0) (type default) (color 0 0 0 0))
   )
+  (wire (pts (xy 160.02 100.33) (xy 160.02 101.6))
+    (stroke (width 0) (type default) (color 0 0 0 0))
+  )
   (wire (pts (xy 153.67 100.33) (xy 160.02 100.33))
     (stroke (width 0) (type default) (color 0 0 0 0))
   )
-  (wire (pts (xy 160.02 100.33) (xy 160.02 101.6))
-    (stroke (width 0) (type default) (color 0 0 0 0))
-  )
   (wire (pts (xy 160.02 101.6) (xy 166.37 101.6))
     (stroke (width 0) (type default) (color 0 0 0 0))
   )
+  (wire (pts (xy 175.26 88.9) (xy 177.8 88.9))
+    (stroke (width 0) (type default) (color 0 0 0 0))
+  )
+  (wire (pts (xy 161.29 88.9) (xy 161.29 82.55))
+    (stroke (width 0) (type default) (color 0 0 0 0))
+  )
   (wire (pts (xy 161.29 82.55) (xy 175.26 82.55))
     (stroke (width 0) (type default) (color 0 0 0 0))
@@
     (stroke (width 0) (type default) (color 0 0 0 0))
   )
-  (wire (pts (xy 161.29 88.9) (xy 161.29 82.55))
-    (stroke (width 0) (type default) (color 0 0 0 0))
-  )
-  (wire (pts (xy 175.26 88.9) (xy 177.8 88.9))
-    (stroke (width 0) (type default) (color 0 0 0 0))
-  )
   (wire (pts (xy 177.8 97.79) (xy 177.8 93.98))
     (stroke (width 0) (type default) (color 0 0 0 0))
@@
     (stroke (width 0) (type default) (color 0 0 0 0))
   )
+  (polyline (pts (xy 87.63 67.31) (xy 133.35 67.31))
+    (stroke (width 0) (type default) (color 0 0 0 0))
+  )
+  (polyline (pts (xy 133.35 67.31) (xy 133.35 127))
+    (stroke (width 0) (type default) (color 0 0 0 0))
+  )
+  (polyline (pts (xy 133.35 127) (xy 87.63 127))
+    (stroke (width 0) (type default) (color 0 0 0 0))
+  )
   (polyline (pts (xy 87.63 127) (xy 87.63 67.31))
     (stroke (width 0) (type default) (color 0 0 0 0))
   )
-  (polyline (pts (xy 87.63 67.31) (xy 133.35 67.31))
-    (stroke (width 0) (type default) (color 0 0 0 0))
-  )
-  (polyline (pts (xy 133.35 127) (xy 87.63 127))
-    (stroke (width 0) (type default) (color 0 0 0 0))
-  )
-  (polyline (pts (xy 133.35 67.31) (xy 133.35 127))
-    (stroke (width 0) (type default) (color 0 0 0 0))
-  )
   (wire (pts (xy 113.03 109.22) (xy 118.11 109.22))
     (stroke (width 0) (type default) (color 0 0 0 0))
@@
     (stroke (width 0) (type default) (color 0 0 0 0))
   )
+  (wire (pts (xy 153.67 109.22) (xy 160.02 109.22))
+    (stroke (width 0) (type default) (color 0 0 0 0))
+  )
   (wire (pts (xy 160.02 110.49) (xy 166.37 110.49))
     (stroke (width 0) (type default) (color 0 0 0 0))
   )
   (wire (pts (xy 160.02 109.22) (xy 160.02 110.49))
-    (stroke (width 0) (type default) (color 0 0 0 0))
-  )
-  (wire (pts (xy 153.67 109.22) (xy 160.02 109.22))
     (stroke (width 0) (type default) (color 0 0 0 0))
   )
@@
     (effects (font (size 1.27 1.27)) (justify left bottom))
   )
-  (symbol (lib_id "ao_symbols:R_POT") (at 166.37 106.68 180) (unit 1)
+  (symbol (lib_name "R_POT_1") (lib_id "ao_symbols:R_POT") (at 166.37 106.68 0) (mirror y) (unit 1)
     (in_bom yes) (on_board yes) (fields_autoplaced)
-    (property "Reference" "RV3" (id 0) (at 168.148 105.7715 0)
-      (effects (font (size 1.27 1.27)) (justify right))
-    )
-    (property "Value" "100k" (id 1) (at 168.148 108.5466 0)
+    (property "Reference" "RV3" (id 0) (at 168.148 106.1271 0)
+      (effects (font (size 1.27 1.27)) (justify right))
+    )
+    (property "Value" "100k" (id 1) (at 168.148 108.9022 0)
       (effects (font (size 1.27 1.27)) (justify right))
     )
@@
     (pin "3")
   )
-  (symbol (lib_id "ao_symbols:R_POT") (at 166.37 97.79 180) (unit 1)
+  (symbol (lib_name "R_POT_2") (lib_id "ao_symbols:R_POT") (at 166.37 97.79 0) (mirror y) (unit 1)
     (in_bom yes) (on_board yes) (fields_autoplaced)
-    (property "Reference" "RV2" (id 0) (at 168.148 96.8815 0)
-      (effects (font (size 1.27 1.27)) (justify right))
-    )
-    (property "Value" "100k" (id 1) (at 168.148 99.6566 0)
+    (property "Reference" "RV2" (id 0) (at 168.148 97.2371 0)
+      (effects (font (size 1.27 1.27)) (justify right))
+    )
+    (property "Value" "100k" (id 1) (at 168.148 100.0122 0)
       (effects (font (size 1.27 1.27)) (justify right))
     )
@@
     (pin "T")
   )
-  (symbol (lib_id "ao_symbols:R_POT") (at 166.37 88.9 180) (unit 1)
+  (symbol (lib_name "R_POT_3") (lib_id "ao_symbols:R_POT") (at 166.37 88.9 0) (mirror y) (unit 1)
     (in_bom yes) (on_board yes) (fields_autoplaced)
-    (property "Reference" "RV1" (id 0) (at 168.148 87.9915 0)
-      (effects (font (size 1.27 1.27)) (justify right))
-    )
-    (property "Value" "100k" (id 1) (at 168.148 90.7666 0)
+    (property "Reference" "RV1" (id 0) (at 168.148 88.3471 0)
+      (effects (font (size 1.27 1.27)) (justify right))
+    )
+    (property "Value" "100k" (id 1) (at 168.148 91.1222 0)
       (effects (font (size 1.27 1.27)) (justify right))
     )
@@
     (pin "3")
   )
-  (symbol (lib_id "ao_symbols:R_POT") (at 181.61 88.9 180) (unit 1)
+  (symbol (lib_name "R_POT_4") (lib_id "ao_symbols:R_POT") (at 181.61 88.9 0) (mirror y) (unit 1)
     (in_bom yes) (on_board yes) (fields_autoplaced)
-    (property "Reference" "RV7" (id 0) (at 183.388 87.9915 0)
-      (effects (font (size 1.27 1.27)) (justify right))
-    )
-    (property "Value" "100k" (id 1) (at 183.388 90.7666 0)
+    (property "Reference" "RV7" (id 0) (at 183.388 88.3471 0)
+      (effects (font (size 1.27 1.27)) (justify right))
+    )
+    (property "Value" "100k" (id 1) (at 183.388 91.1222 0)
       (effects (font (size 1.27 1.27)) (justify right))
     )
@@
     (pin "2")
   )
-  (symbol (lib_id "ao_symbols:R_POT") (at 181.61 106.68 180) (unit 1)
+  (symbol (lib_name "R_POT_5") (lib_id "ao_symbols:R_POT") (at 181.61 106.68 0) (mirror y) (unit 1)
     (in_bom yes) (on_board yes) (fields_autoplaced)
-    (property "Reference" "RV9" (id 0) (at 183.388 105.7715 0)
-      (effects (font (size 1.27 1.27)) (justify right))
-    )
-    (property "Value" "100k" (id 1) (at 183.388 108.5466 0)
+    (property "Reference" "RV9" (id 0) (at 183.388 106.1271 0)
+      (effects (font (size 1.27 1.27)) (justify right))
+    )
+    (property "Value" "100k" (id 1) (at 183.388 108.9022 0)
       (effects (font (size 1.27 1.27)) (justify right))
     )
@@
     (pin "2")
   )
-  (symbol (lib_id "ao_symbols:R_POT") (at 181.61 97.79 180) (unit 1)
+  (symbol (lib_id "ao_symbols:R_POT") (at 181.61 97.79 0) (mirror y) (unit 1)
     (in_bom yes) (on_board yes) (fields_autoplaced)
-    (property "Reference" "RV8" (id 0) (at 183.388 96.8815 0)
-      (effects (font (size 1.27 1.27)) (justify right))
-    )
-    (property "Value" "100k" (id 1) (at 183.388 99.6566 0)
-      (effects (font (size 1.27 1.27)) (justify right))
-    )
+    (property "Reference" "RV8" (id 0) (at 183.388 97.2371 0)
+      (effects (font (size 1.27 1.27)) (justify right))
+    )
+    (property "Value" "100k" (id 1) (at 183.388 100.0122 0)
+      (effects (font (size 1.27 1.27)) (justify right))
+    )

Commit message: rm first design; add new holes image
Parts:
- removed J11: 2_pin_Molex_header, ao_tht:Molex_KK-254_AE-6410-02A_1x02_P2.54mm_Vertical, symbol ao_symbols:2_pin_Molex_header
- removed J15: 2_pin_Molex_connector, symbol ao_symbols:2_pin_Molex_connector
- removed J6: AudioJack2, ao_tht:Jack_6.35mm_PJ_629HAN_slots, symbol Connector:AudioJack2
- removed RV7, RV8, RV9: 100k, ao_tht:Potentiometer_Alpha_RD901F-40-00D_Single_Vertical_centered, symbol ao_symbols:R_POT
- renumbered J7 to J1, J12 to J2, J8 to J3, J13 to J4, J10 to J5, J14 to J6, RV2 to RV3, RV3 to RV5
Other:
- sheet Main PCB ports: added none; removed OUT B
- note removed: "Fit either 16 mm or 9 mm pots"
- moved on the sheet: J2, J4, J6, RV1, RV3, RV5
